File: CircuitDesing/Sensores/embebidos.kicad_sch (KiCad schematic)
At the start: 12 parts, among them J1 Conn_01x03_Male

Commit message: Programacion
Connections:
- net 5v: now also RIEGO1.7
- net GND: now also COMUNICACION1.8, RIEGO1.8
- no-connect marks 3 -> 0
Other:
- note removed: "Pantalla HMI"
Changed lines of the file:
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@@
   (junction (at 133.35 135.89) (diameter 0) (color 0 0 0 0)
   )
-  (no_connect (at 87.63 129.54))
-  (no_connect (at 87.63 132.08))
-  (no_connect (at 179.07 138.43))
   (wire (pts (xy 132.08 135.89) (xy 133.35 135.89))
     (stroke (width 0) (type default) (color 0 0 0 0))
@@
   )
   (wire (pts (xy 30.48 25.4) (xy 43.18 25.4))
+    (stroke (width 0) (type default) (color 0 0 0 0))
+  )
+  (wire (pts (xy 87.63 135.89) (xy 87.63 132.08))
     (stroke (width 0) (type default) (color 0 0 0 0))
   )
@@
   (text "Grupo sensores: 6 pines GPIO\nGrupo comunicación: 6 pines GPIO\nGrupo actuadore (tem,hum,ilu): 2 pines GPIO + 1 I2C\nGrupo riego: 5 pines GPIO\nGrupo cámara: Bluetooth\n\n\n"
     (at 210.82 78.74 0)
-    (effects (font (size 1.27 1.27)) (justify left bottom))
-  )
-  (text "Pantalla HMI" (at 137.16 113.03 0)
     (effects (font (size 1.27 1.27)) (justify left bottom))
   )
@@
     (property "Intersheet References" "${INTERSHEET_REFS}" (id 0) (at 205.7945 72.3106 0)
       (effects (font (size 1.27 1.27)) (justify left) hide)
+    )
+  )
+  (global_label "5v" (shape input) (at 87.63 129.54 180) (fields_autoplaced)
+    (effects (font (size 1.27 1.27)) (justify right))
+    (property "Intersheet References" "${INTERSHEET_REFS}" (id 0) (at 83.0398 129.6194 0)
+      (effects (font (size 1.27 1.27)) (justify right) hide)
     )
   )
@@
     (pin "8")
   )
+  (symbol (lib_id "power:GND") (at 87.63 135.89 270) (unit 1)
+    (in_bom yes) (on_board yes)
+    (property "Reference" "#PWR0104" (id 0) (at 81.28 135.89 0)
+      (effects (font (size 1.27 1.27)) hide)
+    )
+    (property "Value" "GND" (id 1) (at 81.28 135.89 90)
+      (effects (font (size 1.27 1.27)) (justify left))
+    )
+    (property "Footprint" "" (id 2) (at 87.63 135.89 0)
+      (effects (font (size 1.27 1.27)) hide)
+    )
+    (property "Datasheet" "" (id 3) (at 87.63 135.89 0)
+      (effects (font (size 1.27 1.27)) hide)
+    )
+    (pin "1")
+  )
+  (symbol (lib_id "power:GND") (at 179.07 138.43 270) (unit 1)
+    (in_bom yes) (on_board yes)
+    (property "Reference" "#PWR0103" (id 0) (at 172.72 138.43 0)
+      (effects (font (size 1.27 1.27)) hide)
+    )
+    (property "Value" "GND" (id 1) (at 172.72 138.43 90)
+      (effects (font (size 1.27 1.27)) (justify left))
+    )
+    (property "Footprint" "" (id 2) (at 179.07 138.43 0)
+      (effects (font (size 1.27 1.27)) hide)
+    )
+    (property "Datasheet" "" (id 3) (at 179.07 138.43 0)
+      (effects (font (size 1.27 1.27)) hide)
+    )
+    (pin "1")
+  )
   (symbol (lib_id "Device:R") (at 139.7 130.81 0) (unit 1)
     (in_bom yes) (on_board yes)
@@
       (reference "#PWR0102") (unit 1) (value "GND") (footprint "")
     )
+    (path "/35df1bd9-dbec-4b54-8a6e-ca33369608f2"
+      (reference "#PWR0103") (unit 1) (value "GND") (footprint "")
+    )
+    (path "/30c080ee-762a-4f39-942e-188646f40f46"
+      (reference "#PWR0104") (unit 1) (value "GND") (footprint "")
+    )
     (path "/572805be-d728-451f-a777-de266376eb34"
