File: CircuitDesing/Sensores/Con_digital.kicad_sch (KiCad schematic)
At the start: 6 parts, among them Q1 BSS138, Q2 BSS138

Commit message: Ruteo2.0
Parts:
- renumbered Q1 to Q2, Q2 to Q3, R1 to R4, R2 to R5, R3 to R6, R4 to R7
Changed lines of the file:
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@@
   (symbol (lib_id "Device:R") (at 153.67 82.55 0) (unit 1)
     (in_bom yes) (on_board yes) (fields_autoplaced)
-    (property "Reference" "R4" (id 0) (at 156.21 81.2799 0)
+    (property "Reference" "R7" (id 0) (at 156.21 81.2799 0)
       (effects (font (size 1.27 1.27)) (justify left))
     )
@@
   (symbol (lib_id "Device:R") (at 80.01 82.55 0) (unit 1)
     (in_bom yes) (on_board yes) (fields_autoplaced)
-    (property "Reference" "R1" (id 0) (at 82.55 81.2799 0)
+    (property "Reference" "R4" (id 0) (at 82.55 81.2799 0)
       (effects (font (size 1.27 1.27)) (justify left))
     )
@@
   (symbol (lib_id "Transistor_FET:BSS138") (at 88.9 92.71 270) (unit 1)
     (in_bom yes) (on_board yes) (fields_autoplaced)
-    (property "Reference" "Q1" (id 0) (at 88.9 100.33 90))
+    (property "Reference" "Q2" (id 0) (at 88.9 100.33 90))
     (property "Value" "BSS138" (id 1) (at 88.9 102.87 90))
     (property "Footprint" "Package_TO_SOT_SMD:SOT-23" (id 2) (at 86.995 97.79 0)
@@
   (symbol (lib_id "Device:R") (at 135.89 82.55 0) (unit 1)
     (in_bom yes) (on_board yes) (fields_autoplaced)
-    (property "Reference" "R3" (id 0) (at 138.43 81.2799 0)
+    (property "Reference" "R6" (id 0) (at 138.43 81.2799 0)
       (effects (font (size 1.27 1.27)) (justify left))
     )
@@
   (symbol (lib_id "Transistor_FET:BSS138") (at 144.78 92.71 270) (unit 1)
     (in_bom yes) (on_board yes) (fields_autoplaced)
-    (property "Reference" "Q2" (id 0) (at 144.78 100.33 90))
+    (property "Reference" "Q3" (id 0) (at 144.78 100.33 90))
     (property "Value" "BSS138" (id 1) (at 144.78 102.87 90))
     (property "Footprint" "Package_TO_SOT_SMD:SOT-23" (id 2) (at 142.875 97.79 0)
@@
   (symbol (lib_id "Device:R") (at 97.79 82.55 0) (unit 1)
     (in_bom yes) (on_board yes) (fields_autoplaced)
-    (property "Reference" "R2" (id 0) (at 100.33 81.2799 0)
+    (property "Reference" "R5" (id 0) (at 100.33 81.2799 0)
       (effects (font (size 1.27 1.27)) (justify left))
     )
