File: CircuitDesing/Sensores/Esp32Schematic.kicad_sch (KiCad schematic)
At the start: 9 parts, among them SW1 SW_Push, SW2 SW_Push, U1 ESP32-WROOM-32

Commit message: Ruteo listo
Parts:
- renumbered SW2 to BOOT1, SW1 to EN1
Changed lines of the file:
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@@
+    (stroke (width 0) (type default) (color 0 0 0 0))
+  )
+  (wire (pts (xy 83.82 135.89) (xy 92.71 135.89))
     (stroke (width 0) (type default) (color 0 0 0 0))
   )
@@
     (stroke (width 0) (type default) (color 0 0 0 0))
   )
+  (wire (pts (xy 86.36 140.97) (xy 83.82 140.97))
+    (stroke (width 0) (type default) (color 0 0 0 0))
+  )
   (wire (pts (xy 105.41 69.85) (xy 119.38 69.85))
     (stroke (width 0) (type default) (color 0 0 0 0))
@@
     (stroke (width 0) (type default) (color 0 0 0 0))
   )
+  (wire (pts (xy 83.82 140.97) (xy 83.82 142.24))
+    (stroke (width 0) (type default) (color 0 0 0 0))
+  )
   (wire (pts (xy 119.38 69.85) (xy 119.38 78.74))
     (stroke (width 0) (type default) (color 0 0 0 0))
@@
   )
   (wire (pts (xy 66.04 77.47) (xy 68.58 77.47))
-    (stroke (width 0) (type default) (color 0 0 0 0))
-  )
-  (wire (pts (xy 83.82 137.16) (xy 83.82 135.89))
     (stroke (width 0) (type default) (color 0 0 0 0))
   )
@@
     (effects (font (size 1.27 1.27)) (justify left bottom))
   )
+  (label "gnd" (at 92.71 135.89 0)
+    (effects (font (size 1.27 1.27)) (justify left bottom))
+  )
   (label "BOOT" (at 105.41 69.85 0)
     (effects (font (size 1.27 1.27)) (justify left bottom))
   )
+  (label "gnd" (at 86.36 140.97 0)
+    (effects (font (size 1.27 1.27)) (justify left bottom))
+  )
   (hierarchical_label "IO27" (shape input) (at 99.06 118.11 0)
     (effects (font (size 1.27 1.27)) (justify left))
@@
     (pin "1")
   )
-  (symbol (lib_id "power:GND") (at 83.82 137.16 0) (unit 1)
-    (in_bom yes) (on_board yes) (fields_autoplaced)
-    (property "Reference" "#PWR0103" (id 0) (at 83.82 143.51 0)
-      (effects (font (size 1.27 1.27)) hide)
-    )
-    (property "Value" "GND" (id 1) (at 83.82 142.24 0))
-    (property "Footprint" "" (id 2) (at 83.82 137.16 0)
-      (effects (font (size 1.27 1.27)) hide)
-    )
-    (property "Datasheet" "" (id 3) (at 83.82 137.16 0)
+  (symbol (lib_id "power:GND") (at 83.82 142.24 0) (unit 1)
+    (in_bom yes) (on_board yes) (fields_autoplaced)
+    (property "Reference" "#PWR0103" (id 0) (at 83.82 148.59 0)
+      (effects (font (size 1.27 1.27)) hide)
+    )
+    (property "Value" "GND" (id 1) (at 83.82 147.32 0))
+    (property "Footprint" "" (id 2) (at 83.82 142.24 0)
+      (effects (font (size 1.27 1.27)) hide)
+    )
+    (property "Datasheet" "" (id 3) (at 83.82 142.24 0)
       (effects (font (size 1.27 1.27)) hide)
     )
@@
   (symbol (lib_id "Switch:SW_Push") (at 125.73 69.85 0) (unit 1)
     (in_bom yes) (on_board yes) (fields_autoplaced)
-    (property "Reference" "SW2" (id 0) (at 125.73 62.23 0))
+    (property "Reference" "BOOT1" (id 0) (at 125.73 62.23 0))
     (property "Value" "SW_Push" (id 1) (at 125.73 64.77 0))
     (property "Footprint" "Button_Switch_SMD:SW_Push_1P1T_NO_6x6mm_H9.5mm" (id 2) (at 125.73 64.77 0)
@@
   (symbol (lib_id "Switch:SW_Push") (at 52.07 80.01 0) (unit 1)
     (in_bom yes) (on_board yes) (fields_autoplaced)
-    (property "Reference" "SW1" (id 0) (at 52.07 72.39 0))
+    (property "Reference" "EN1" (id 0) (at 52.07 72.39 0))
     (property "Value" "SW_Push" (id 1) (at 52.07 74.93 0))
     (property "Footprint" "Button_Switch_SMD:SW_Push_1P1T_NO_6x6mm_H9.5mm" (id 2) (at 52.07 74.93 0)

Commit message: Ruteo2.0
Parts:
- renumbered C3 to C1, C1 to C3, R3 to R2
Changed lines of the file:
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@@
   (symbol (lib_id "power:GND") (at 41.91 69.85 270) (unit 1)
     (in_bom yes) (on_board yes) (fields_autoplaced)
-    (property "Reference" "#PWR0101" (id 0) (at 35.56 69.85 0)
+    (property "Reference" "#PWR011" (id 0) (at 35.56 69.85 0)
       (effects (font (size 1.27 1.27)) hide)
     )
@@
   (symbol (lib_id "power:GND") (at 83.82 142.24 0) (unit 1)
     (in_bom yes) (on_board yes) (fields_autoplaced)
-    (property "Reference" "#PWR0103" (id 0) (at 83.82 148.59 0)
+    (property "Reference" "#PWR012" (id 0) (at 83.82 148.59 0)
       (effects (font (size 1.27 1.27)) hide)
     )
@@
   (symbol (lib_id "Device:C_Small") (at 93.98 53.34 90) (mirror x) (unit 1)
     (in_bom yes) (on_board yes)
-    (property "Reference" "C1" (id 0) (at 93.98 59.69 90)
+    (property "Reference" "C3" (id 0) (at 93.98 59.69 90)
       (effects (font (size 1.27 1.27)) (justify right))
     )
@@
   (symbol (lib_id "Device:R") (at 105.41 62.23 0) (unit 1)
     (in_bom yes) (on_board yes) (fields_autoplaced)
-    (property "Reference" "R3" (id 0) (at 107.95 60.9599 0)
+    (property "Reference" "R2" (id 0) (at 107.95 60.9599 0)
       (effects (font (size 1.27 1.27)) (justify left))
     )
@@
   (symbol (lib_id "power:GND") (at 134.62 69.85 90) (unit 1)
     (in_bom yes) (on_board yes) (fields_autoplaced)
-    (property "Reference" "#PWR0102" (id 0) (at 140.97 69.85 0)
+    (property "Reference" "#PWR014" (id 0) (at 140.97 69.85 0)
       (effects (font (size 1.27 1.27)) hide)
     )
@@
   (symbol (lib_id "power:GND") (at 107.95 50.8 90) (unit 1)
     (in_bom yes) (on_board yes)
-    (property "Reference" "#PWR0105" (id 0) (at 114.3 50.8 0)
+    (property "Reference" "#PWR013" (id 0) (at 114.3 50.8 0)
       (effects (font (size 1.27 1.27)) hide)
     )
@@
   (symbol (lib_id "Device:C_Small") (at 52.07 69.85 90) (unit 1)
     (in_bom yes) (on_board yes)
-    (property "Reference" "C3" (id 0) (at 52.0763 63.5 90))
+    (property "Reference" "C1" (id 0) (at 52.0763 63.5 90))
     (property "Value" "1uF" (id 1) (at 52.0763 66.04 90))
     (property "Footprint" "Capacitor_SMD:C_0603_1608Metric_Pad1.08x0.95mm_HandSolder" (id 2) (at 52.07 69.85 0)
